File: hardware/fc-adapter/fc-adapter.kicad_pcb (KiCad board)
At the start: 2 copper layers, 94 x 94 mm, 37 parts, among them J1 XT60 male (from PM02), J10 PM02 lead, J2 ESC signal 3x4, J3 FC link, J5 GPS+ID GH-6, J6 GPS+ID lead, J7 RX GH-4, J8 RX lead, J9 PM02 GH-6, P1 FC VBAT+, P10 M2 ESC-, P11 M3 ESC+, P12 M3 ESC-, P13 M4 ESC+, P14 M4 ESC-, P2 FC VBAT-, P7 M1 ESC+, P8 M1 ESC-, P9 M2 ESC+

Commit message: Fit the second bulk cap (C3 -> C2) for symmetry
Co-Authored-By: Claude Opus 5.5 (1M context) <noreply@anthropic.com>
Claude-Session: https://claude.ai/code/session_01SvgiwfQJ8xhgBPV2g6jXCT
Parts:
- removed C3: DNP 2nd cap, Capacitor_THT:CP_Radial_D12.5mm_P5.00mm
- added C2: 1000uF 35V, Capacitor_THT:CP_Radial_D12.5mm_P5.00mm, F.Cu at (112.5, 102.5)

Commit message: Target OSH Park: 1.6 mm, 1 oz copper, ENIG
OSH Park's 2 oz service is only 0.8 mm, too flexible for a board that
carries the FC; the full-width pours carry the current at 1 oz.

Co-Authored-By: Claude Opus 5.5 (1M context) <noreply@anthropic.com>
Claude-Session: https://claude.ai/code/session_01SvgiwfQJ8xhgBPV2g6jXCT
Other:
- board text added: "1 oz Cu, 1.6 mm FR4"
- board text removed: "2 oz Cu, 2.0 mm FR4"
