File: hardware/fc-adapter/fc-adapter.kicad_sch (KiCad schematic)
At the start: 37 parts, among them J1 XT60 male (from PM02), J10 PM02 lead, J2 ESC signal 3x4, J3 FC link, J5 GPS+ID GH-6, J6 GPS+ID lead, J7 RX GH-4, J8 RX lead, J9 PM02 GH-6, P1 FC VBAT+, P10 M2 ESC-, P11 M3 ESC+, P12 M3 ESC-, P13 M4 ESC+, P14 M4 ESC-, P2 FC VBAT-, P7 M1 ESC+, P8 M1 ESC-, P9 M2 ESC+

Commit message: Fit the second bulk cap (C3 -> C2) for symmetry
Co-Authored-By: Claude Opus 5.5 (1M context) <noreply@anthropic.com>
Claude-Session: https://claude.ai/code/session_01SvgiwfQJ8xhgBPV2g6jXCT
Parts:
- removed C3: DNP 2nd cap, Capacitor_THT:CP_Radial_D12.5mm_P5.00mm, symbol Device:C_Polarized
- added C2: 1000uF 35V, Capacitor_THT:CP_Radial_D12.5mm_P5.00mm, symbol Device:C_Polarized
Connections:
- net GND_ESC: now also C2.2
- net VBAT_ESC: now also C2.1
Other:
- note added: "POWER PATH (rev A): battery -> Holybro PM02 (current sense) -> J1 XT60 -> ESC bus. ESC bus -> M1..M4 ESC pads, P1/P2 (FC VBAT) -> FC VBAT pads. C1, C2: low-ESR, one each side for balance. Signal GND only meets GND_ESC through the FC."
- note removed: "POWER PATH (rev A): battery -> Holybro PM02 (current sense) -> J1 XT60 -> ESC bus. ESC bus -> M1..M4 ESC pads, P1/P2 (FC VBAT) -> FC VBAT pads. C1: low-ESR. Signal GND only meets GND_ESC through the FC."
